File: hardware/eps-re_project/MPPT_Battery_Charger.kicad_sch (KiCad schematic)
At the start: 74 parts, among them Q204 SI7414DN-T1, Q205 SI7414DN-T1, Q5 SI2302, Q6 SI2302, U20 INA199C3DCKR, U22 BQ24650RVAT, U23 SI7414DN-T1, U24 INA199C3DCKR, U25 SI7414DN-T1, U26 LMV321RIYLT, U27 BQ24650RVAT, U28 LMV321RIYLT

Commit message: hardware: Restructuring the circuit, modifying symbols, footprints and other corrections
Parts:
- removed C13, C210, C216, C218, C223: 100nF, symbol Device:C
- removed C212, C23: 10uF, symbol Device:C
- removed C213, C214, C22: 1uF, symbol Device:C
- removed C215: 2.2uF, symbol Device:C
- removed C24: 4.7uF, symbol Device:C
- removed D205: BAT54W, Package_TO_SOT_SMD:SOT-323_SC-70, symbol Diode:BAT54W
- removed D206, D207: LED, symbol Device:LED
- removed D6: PDS1040L-13, DIO_PDS1040L-13, symbol PDS1040L-13:PDS1040L-13
- removed L200, L201: 12uH, symbol Device:L
- removed Q204, Q205, U23, U25: SI7414DN-T1, MOSFET_4DN-T1-E3_VIS, symbol SI7414DN-T1:SI7414DN-T1
- removed Q6: SI2302, SOT23, symbol SI2302:SI2302
- removed R213: 270kR, symbol Device:R
- removed R214: 10R, symbol Device:R
- removed R215: 2R, symbol Device:R
- removed R216: 100K, symbol Device:R
- removed R217, R218: 20kR, symbol Device:R
- removed R220: 5.23k, symbol Device:R
- removed R223: 30.1kR, symbol Device:R
- removed R226, R227: 10k, symbol Device:R
- removed R50: 33mR, symbol Device:R
- removed U20, U24: INA199C3DCKR, DCK0006A_N, symbol INA199C3DCKR:INA199C3DCKR
- removed U27: BQ24650RVAT, RVA16_2P14X2P14, symbol BQ24650RVAT:BQ24650RVAT
- added C11, C12, C3 (x2): 100nF, footprints:C0603C104K5RACTU, symbol C0603C104K5RACTU:C0603C104K5RACTU
- added C14: 2.2uF, footprints:C1210C225K5RACTU, symbol C1210C225K5RACTU:C1210C225K5RACTU
- added C15, C201, C203, C206: 1uF, footprints:C0805C105K5RACTU, symbol C0805C105K5RACTU:C0805C105K5RACTU
- added C200, C208: 10uF, footprints:C1210C106K5RACTU, symbol C1210C106K5RACTU:C1210C106K5RACTU
- added C209: 4700nF, footprints:C1210C475K5RACTU, symbol C1210C475K5RACTU:C1210C475K5RACTU
- added D1, D2: LED, symbol Device:LED_Filled
- added D201: BAT54, footprints:BAT54, symbol BAT54:BAT54
- added D3: PDS1040L-13, footprints:PDS1040L-13, symbol PDS1040L-13:PDS1040L-13
- added L200 (x2): 12uH, footprints:744770112, symbol 744770112:744770112
- added Q24, Q25, Q5, Q6: SI7414DN-T1-E3, footprints:SI7414DN-T1-E3, symbol SI7414DN-T1-E3:SI7414DN-T1-E3
- added Q5: SI2302DDS-T1-GE3, footprints:SI2302DDS-T1-GE3, symbol SI2302DDS-T1-GE3:SI2302DDS-T1-GE3
- added R201: 270k, symbol Device:R_US
- added R202: 10R, symbol Device:R_US
- added R204, R206: 20k, symbol Device:R_US
- added R207: 33m, symbol Device:R_US
- added R209: 5.23k, symbol Device:R_US
- added R31, R36: 10k, symbol Device:R_US
- added R37: 2R, symbol Device:R_US
- added R38: 100k, symbol Device:R_US
- added R39: 30.1k, symbol Device:R_US
- added U22: BQ24650RVAT, footprints:BQ24650RVAT, symbol BQ24650RVAT:BQ24650RVAT
- added U4 (x2): INA199C1DCKR, footprints:INA199C1DCKR, symbol INA199C1DCKR:INA199xxDCK
- C11, C12: footprint (none) -> footprints:C0603C104K5RACTU; symbol Device:C -> C0603C104K5RACTU:C0603C104K5RACTU; automotive (none) -> Yes; automotive grade (none) -> Grade 1; capacitance (none) -> 0.10 μF; category (none) -> Cap; device class L1 (none) -> Passive Components; device class L2 (none) -> Capacitors; device class L3 (none) -> Ceramic Capacitors; digikey description (none) -> CAP CER 0.1UF 50V X7R 0603; digikey part number (none) -> 399-5089-2-ND; height (none) -> 0.87mm; lead free (none) -> Yes; library id (none) -> 73022d3323b2b2b8; manufacturer (none) -> KEMET; material (none) -> Ceramic; mouser part number (none) -> 80-C0603C104K5R7867; package (none) -> 0603; rohs (none) -> Yes; temperature characteristic (none) -> X7R; temperature coefficient (none) -> 30ppm/°C; temperature range high (none) -> +125°C; temperature range low (none) -> -55°C; tolerance (none) -> 0.1; voltage rating (none) -> 50 V
- C14: value 100nF -> 2.2uF; footprint (none) -> footprints:C1210C225K5RACTU; symbol Device:C -> C1210C225K5RACTU:C1210C225K5RACTU; automotive (none) -> No; capacitance (none) -> 2.2uF; category (none) -> Cap; device class L1 (none) -> Passive Components; device class L2 (none) -> Capacitors; device class L3 (none) -> Ceramic Capacitors; digikey description (none) -> CAP CER 2.2UF 50V X7R 1210; digikey part number (none) -> 399-8231-1-ND; height (none) -> 1.4mm; ipc land pattern name (none) -> CAPC320250X125; lead free (none) -> Yes; library id (none) -> dba7d30363bd9f03; manufacturer (none) -> Kemet; material (none) -> Ceramic; mouser description (none) -> Multilayer Ceramic Capacitors MLCC - SMD/SMT 50volts 2.2uF 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; mouser part number (none) -> 80-C1210C225K5R; package (none) -> 1210; rohs (none) -> Yes; temperature characteristic (none) -> X7R; temperature coefficient (none) -> 15%; temperature range high (none) -> +125°C; temperature range low (none) -> -55°C; tolerance (none) -> 10%; voltage rating (none) -> 50V
- C15: value 100nF -> 1uF; footprint (none) -> footprints:C0805C105K5RACTU; symbol Device:C -> C0805C105K5RACTU:C0805C105K5RACTU; capacitance (none) -> 1uF; category (none) -> Cap; device class L1 (none) -> Passive Components; device class L2 (none) -> Capacitors; device class L3 (none) -> Ceramic Capacitors; digikey description (none) -> CAP CER 1UF 50V X7R 0805; digikey part number (none) -> 399-7409-2-ND; height (none) -> 1.4mm; ipc land pattern name (none) -> CAPC200125X787; lead free (none) -> yes; library id (none) -> ac83af3950e2a3c3; manufacturer (none) -> Kemet; material (none) -> Ceramic; mouser description (none) -> Multilayer Ceramic Capacitors MLCC - SMD/SMT 1uF 50 Volts 1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; mouser part number (none) -> 80-C0805C105K5R; package (none) -> 0805 (2012 metric); rohs (none) -> yes; standoff height (none) -> 0mm; temperature characteristic (none) -> X7R; temperature range high (none) -> +125°C; temperature range low (none) -> -55°C; tolerance (none) -> 10%; voltage rating (none) -> 50V
- C16: value 1uF -> 100nF; footprint (none) -> footprints:C0603C104K5RACTU; symbol Device:C -> C0603C104K5RACTU:C0603C104K5RACTU; automotive (none) -> Yes; automotive grade (none) -> Grade 1; capacitance (none) -> 0.10 μF; category (none) -> Cap; device class L1 (none) -> Passive Components; device class L2 (none) -> Capacitors; device class L3 (none) -> Ceramic Capacitors; digikey description (none) -> CAP CER 0.1UF 50V X7R 0603; digikey part number (none) -> 399-5089-2-ND; height (none) -> 0.87mm; lead free (none) -> Yes; library id (none) -> 73022d3323b2b2b8; manufacturer (none) -> KEMET; material (none) -> Ceramic; mouser part number (none) -> 80-C0603C104K5R7867; package (none) -> 0603; rohs (none) -> Yes; temperature characteristic (none) -> X7R; temperature coefficient (none) -> 30ppm/°C; temperature range high (none) -> +125°C; temperature range low (none) -> -55°C; tolerance (none) -> 0.1; voltage rating (none) -> 50 V
- C200, C208: footprint (none) -> footprints:C1210C106K5RACTU; symbol Device:C -> C1210C106K5RACTU:C1210C106K5RACTU; automotive (none) -> No; capacitance (none) -> 10uF; category (none) -> Cap; device class L1 (none) -> Passive Components; device class L2 (none) -> Capacitors; device class L3 (none) -> Ceramic Capacitors; digikey description (none) -> CAP CER 10UF 50V X7R 1210; digikey part number (none) -> 399-11629-1-ND; height (none) -> 2.8mm; ipc land pattern name (none) -> CAPC320250X250; lead free (none) -> Yes; library id (none) -> 80b9cd679ce51e4b; manufacturer (none) -> KEMET; material (none) -> Ceramic; mouser description (none) -> Multilayer Ceramic Capacitors MLCC - SMD/SMT 50volts 10uF 1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; mouser part number (none) -> 80-C1210C106K5R; package (none) -> 1210; rohs (none) -> Yes; temperature characteristic (none) -> X7R; temperature coefficient (none) -> 15%; temperature range high (none) -> +125°C; temperature range low (none) -> -55°C; tolerance (none) -> 10%; voltage rating (none) -> 50V
- C201, C203, C206: footprint (none) -> footprints:C0805C105K5RACTU; symbol Device:C -> C0805C105K5RACTU:C0805C105K5RACTU; capacitance (none) -> 1uF; category (none) -> Cap; device class L1 (none) -> Passive Components; device class L2 (none) -> Capacitors; device class L3 (none) -> Ceramic Capacitors; digikey description (none) -> CAP CER 1UF 50V X7R 0805; digikey part number (none) -> 399-7409-2-ND; height (none) -> 1.4mm; ipc land pattern name (none) -> CAPC200125X787; lead free (none) -> yes; library id (none) -> ac83af3950e2a3c3; manufacturer (none) -> Kemet; material (none) -> Ceramic; mouser description (none) -> Multilayer Ceramic Capacitors MLCC - SMD/SMT 1uF 50 Volts 1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; mouser part number (none) -> 80-C0805C105K5R; package (none) -> 0805 (2012 metric); rohs (none) -> yes; standoff height (none) -> 0mm; temperature characteristic (none) -> X7R; temperature range high (none) -> +125°C; temperature range low (none) -> -55°C; tolerance (none) -> 10%; voltage rating (none) -> 50V
- C209: value 4.7uF -> 4700nF; footprint (none) -> footprints:C1210C475K5RACTU; symbol Device:C -> C1210C475K5RACTU:C1210C475K5RACTU; automotive (none) -> No; capacitance (none) -> 4.7uF; category (none) -> Cap; device class L1 (none) -> Passive Components; device class L2 (none) -> Capacitors; device class L3 (none) -> Ceramic Capacitors; digikey description (none) -> CAP CER 4.7UF 50V X7R 1210; digikey part number (none) -> 399-6785-1-ND; height (none) -> 2.8mm; ipc land pattern name (none) -> CAPC320250X250; lead free (none) -> Yes; library id (none) -> 42a2a19c5d7551bb; manufacturer (none) -> Kemet; material (none) -> Ceramic; mouser description (none) -> Multilayer Ceramic Capacitors MLCC - SMD/SMT 50volts 4.7uF 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; mouser part number (none) -> 80-C1210C475K5R; package (none) -> 1210; rohs (none) -> Yes; temperature characteristic (none) -> X7R; temperature range high (none) -> +125°C; temperature range low (none) -> -55°C; tolerance (none) -> 10%; voltage rating (none) -> 50V
- C221: value 100uF -> 100nF; footprint (none) -> footprints:C0603C104K5RACTU; symbol Device:C -> C0603C104K5RACTU:C0603C104K5RACTU; automotive (none) -> Yes; automotive grade (none) -> Grade 1; capacitance (none) -> 0.10 μF; category (none) -> Cap; device class L1 (none) -> Passive Components; device class L2 (none) -> Capacitors; device class L3 (none) -> Ceramic Capacitors; digikey description (none) -> CAP CER 0.1UF 50V X7R 0603; digikey part number (none) -> 399-5089-2-ND; height (none) -> 0.87mm; lead free (none) -> Yes; library id (none) -> 73022d3323b2b2b8; manufacturer (none) -> KEMET; material (none) -> Ceramic; mouser part number (none) -> 80-C0603C104K5R7867; package (none) -> 0603; rohs (none) -> Yes; temperature characteristic (none) -> X7R; temperature coefficient (none) -> 30ppm/°C; temperature range high (none) -> +125°C; temperature range low (none) -> -55°C; tolerance (none) -> 0.1; voltage rating (none) -> 50 V
- D1, D2: symbol Device:LED -> Device:LED_Filled
- D201: value BAT54W -> BAT54; footprint Package_TO_SOT_SMD:SOT-323_SC-70 -> footprints:BAT54; symbol Diode:BAT54W -> BAT54:BAT54; Height (none) -> 1.1; Manufacturer_Name (none) -> Rectron; Manufacturer_Part_Number (none) -> BAT54; Mouser Part Number (none) -> 583-BAT54; Mouser Price/Stock (none) -> https://www.mouser.co.uk/ProductDetail/Rectron/BAT54?qs=7pE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
- D3: footprint DIO_PDS1040L-13 -> footprints:PDS1040L-13
- Q5: value SI2302 -> SI2302DDS-T1-GE3; footprint SOT23 -> footprints:SI2302DDS-T1-GE3; symbol SI2302:SI2302 -> SI2302DDS-T1-GE3:SI2302DDS-T1-GE3; Height (none) -> 1.12; Manufacturer_Name (none) -> Vishay; Manufacturer_Part_Number (none) -> SI2302DDS-T1-GE3; Mouser Part Number (none) -> 78-SI2302DDS-T1-GE3; Mouser Price/Stock (none) -> https://www.mouser.co.uk/ProductDetail/Vishay-Semiconductor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
- R200: value 25mR -> 25m; symbol Device:R -> Device:R_US
- R201: value 270kR -> 270k; symbol Device:R -> Device:R_US
- R202, R209, R31, R36: symbol Device:R -> Device:R_US
- R204, R206: value 20kR -> 20k; symbol Device:R -> Device:R_US
- R207: value 33mR -> 33m; symbol Device:R -> Device:R_US
- R208: value 20mR -> 20m; symbol Device:R -> Device:R_US
- R221: value 30kR -> 30k; symbol Device:R -> Device:R_US
- R222: value 24kR -> 24k; symbol Device:R -> Device:R_US
- R224: value 8.2kR -> 8.2k; symbol Device:R -> Device:R_US
- R225: value 7.5kR -> 7.5k; symbol Device:R -> Device:R_US
- R37: value 25mR -> 2R; symbol Device:R -> Device:R_US
- R38: value 25mR -> 100k; symbol Device:R -> Device:R_US
- R39: value 30.1kR -> 30.1k; symbol Device:R -> Device:R_US
- U22: footprint RVA16_2P14X2P14 -> footprints:BQ24650RVAT
- U26, U28: footprint SOT23-5_STM -> footprints:LMV321RIYLT; symbol LM321RIYLT:LMV321RIYLT -> LMV321RIYLT:LMV321RIYLT
Connections:
- net AMUX0: now also U4.6 (OUT)
- net AMUX1: now also U28.1, U28.4 (-)
- net AMUX2: now also U4.6 (OUT)
- net AMUX3: no longer R222.2, R225.1, U26.3 (NON-INVERTING_INPUT)
- net BC_B_TS: now also R209.2, R39.1, U22.4 (TS)
- net BC_VFB: now also U22.8 (VFB)
- net VBC_IN: now also R31.2, R36.2
- net VBC_N: now also D3.1, D3.2, R201.1, R37.1, U4.5 (IN-)
- net VIN: now also U4.5 (IN-)
- net VPANELS: now also C3.1, U4.3 (V+), U4.4 (IN+)
- net at C200.1, C201.1, D3.3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: now also Q5.5-6-7-8 (D)
- net VCC1: now reaches C203.1, R202.2, U22.1 (VCC)
- net VREF1: now reaches C15.1, R209.1, U22.6 (VREF), U22.7 (TERM_EN)
- net VBC_OUT: now reaches C11.2, C208.1, C209.1, R207.2, R208.2, U22.9 (SRN)
- net VBC_OUT: now also C11.2, C208.1, C209.1, C3.1, R207.2, U22.9 (SRN), U4.3 (V+), U4.4 (IN+)
- net REGN1: now reaches C206.1, D201.1, U22.12 (REGN)
- net BTST1: now reaches D201.2
- net BTST1: now also C12.1, U22.16 (BTST)
- net PH1: now reaches C12.2, U22.14 (PH)
- net at C11.1, R207.1, U22.10 (SRP): now also L200.2
- net at U22.15 (HIDRV): now also Q5.4 (G)
- net at U22.13 (LODRV): now also Q6.4 (G)
- net BC_A_EN renamed BC_A_~{EN}
- net Earth renamed GND
- net GND: now also C14.2, C15.2, C200.2, C201.2, C203.2, C206.2, C208.2, C209.2, C3.2, C3.2, Q25.1 (S), Q25.2 (S), Q25.3 (S), Q5.2 (S), Q6.1 (S), Q6.2 (S), Q6.3 (S), R206.2, R38.2, R39.2, U22.11 (GND), U22.17 (EPAD), U4.1 (REF), U4.1 (REF), U4.2 (GND), U4.2 (GND)
- new net: C200.1, C201.1, D3.3, Q24.5-6-7-8 (D), R202.1
- new net: L200.1, Q5.1 (S), Q5.2 (S), Q5.3 (S), Q6.5-6-7-8 (D)
- new net: D2.2 (A), R36.1
- new net: C11.1, L200.2, R207.1, U22.10 (SRP)
- new net: Q5.3 (D), R201.2, R204.1, U22.2 (MPPSET)
- new net: R204.2, R206.1
- new net: Q25.4 (G), U22.13 (LODRV)
- new net: L200.1, Q24.1 (S), Q24.2 (S), Q24.3 (S), Q25.5-6-7-8 (D)
- new net: R222.2, R225.1, U26.3 (+)
- new net: Q24.4 (G), U22.15 (HIDRV)
- new net: D2.1 (K), U22.3 (STAT1)
- new net: D1.1 (K), U22.5 (STAT2)
- new net: R209.1, U22.7 (TERM_EN)
- new net: C14.1, R37.2
- new net: D1.2 (A), R31.1
- new net BC_B_~{EN}: Q5.1 (G), R38.1
- new net BTST2: C12.1, D201.2, U22.16 (BTST)
- new net PH2: C12.2, U22.14 (PH)
- new net REGN2: C206.1, D201.1, U22.12 (REGN)
- new net VCC2: C203.1, R202.2, U22.1 (VCC)
- new net VREF2: C15.1, U22.6 (VREF)
- now unconnected: D201.3 (K)
Other:
- moved on the sheet: C11, C12, C14, C15, C16, C200, C201, C203, C206, C208, C209, C221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
