File: hardware/5V0_Load_Converters.kicad_sch (KiCad schematic)
At the start: 73 parts, among them J19 61300311121, Q2 SI2302DDS-T1-GE3, Q26 EPC2016C, Q27 EPC2016C, U21 INA199C3DCKR, U30 LTC3833EUDC-TRPBF

Commit message: hardware: starting the pcb project
Parts:
- removed Q2 (x2): SI2302DDS-T1-GE3, footprints:SI2302DDS-T1-GE3, symbol SI2302DDS-T1-GE3:SI2302DDS-T1-GE3
- added Q8 (x2): SI2302DDS-T1-GE3, footprints:SI2302DDS-T1-GE3, symbol SI2302DDS-T1-GE3:SI2302DDS-T1-GE3
Connections:
- net 5V0_A_~{EN}: now also Q8.1 (G)
- net 5V0_B_~{EN}: now also Q8.1 (G)
- net GND: now also Q8.2 (S), Q8.2 (S)
- net at U30.7 (RUN): now also Q8.3 (D) (x2)
Changed lines of the file:
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@@
-    )
-  )
-  (symbol (lib_id "SI2302DDS-T1-GE3:SI2302DDS-T1-GE3") (at 115.57 69.85 0) (unit 1)
-    (in_bom yes) (on_board yes) (dnp no)
-    (property "Reference" "Q2" (at 114.808 60.198 0)
-      (effects (font (size 1.27 1.27)) (justify left))
-    )
-    (property "Value" "SI2302DDS-T1-GE3" (at 99.568 62.738 0)
-      (effects (font (size 1.27 1.27)) (justify left))
-    )
-    (property "Footprint" "footprints:SI2302DDS-T1-GE3" (at 104.14 104.14 0) (show_name)
-      (effects (font (size 1.27 1.27)) (justify left top) hide)
-    )
-    (property "Datasheet" "http://www.vishay.com/docs/63653/si2302dds.pdf" (at 91.186 106.934 0) (show_name)
-      (effects (font (size 1.27 1.27)) (justify left top) hide)
-    )
-    (property "Height" "1.12" (at 127 468.58 0)
-      (effects (font (size 1.27 1.27)) (justify left top) hide)
-    )
-    (property "Mouser Part Number" "78-SI2302DDS-T1-GE3" (at 127 568.58 0)
-      (effects (font (size 1.27 1.27)) (justify left top) hide)
-    )
-    (property "Mouser Price/Stock" "https://www.mouser.co.uk/ProductDetail/Vishay-Semiconductors/SI2302DDS-T1-GE3?qs=MxnWX8BLHKdaCSNWhg%252BxLA%3D%3D" (at 127 668.58 0)
-      (effects (font (size 1.27 1.27)) (justify left top) hide)
-    )
-    (property "Manufacturer_Name" "Vishay" (at 127 768.58 0)
-      (effects (font (size 1.27 1.27)) (justify left top) hide)
-    )
-    (property "Manufacturer_Part_Number" "SI2302DDS-T1-GE3" (at 127 868.58 0)
-      (effects (font (size 1.27 1.27)) (justify left top) hide)
-    )
-    (pin "1")
-    (pin "2")
-    (pin "3")
-    (instances
-      (project "eps-re_project"
-        (path "/2eebaa11-d7ed-4bfd-bc8e-988f68654d29/6f34948c-43a8-4614-b8ed-90c5b6b9b243"
-          (reference "Q2") (unit 1)
-        )
-        (path "/2eebaa11-d7ed-4bfd-bc8e-988f68654d29/6cd5fe02-9b19-49bf-9109-b0a2c2f10c14"
-          (reference "Q1") (unit 1)
-        )
-      )
     )
   )
@@
     )
   )
-  (symbol (lib_id "SI2302DDS-T1-GE3:SI2302DDS-T1-GE3") (at 115.57 170.18 0) (unit 1)
+  (symbol (lib_id "SI2302DDS-T1-GE3:SI2302DDS-T1-GE3") (at 115.57 69.85 0) (unit 1)
     (in_bom yes) (on_board yes) (dnp no)
-    (property "Reference" "Q2" (at 115.57 172.72 0)
-      (effects (font (size 1.27 1.27)) (justify left))
-    )
-    (property "Value" "SI2302DDS-T1-GE3" (at 100.33 175.26 0)
-      (effects (font (size 1.27 1.27)) (justify left))
-    )
-    (property "Footprint" "footprints:SI2302DDS-T1-GE3" (at 104.14 204.47 0) (show_name)
-      (effects (font (size 1.27 1.27)) (justify left top) hide)
-    )
-    (property "Datasheet" "http://www.vishay.com/docs/63653/si2302dds.pdf" (at 91.186 207.264 0) (show_name)
-      (effects (font (size 1.27 1.27)) (justify left top) hide)
-    )
-    (property "Height" "1.12" (at 127 568.91 0)
-      (effects (font (size 1.27 1.27)) (justify left top) hide)
-    )
-    (property "Mouser Part Number" "78-SI2302DDS-T1-GE3" (at 127 668.91 0)
-      (effects (font (size 1.27 1.27)) (justify left top) hide)
-    )
-    (property "Mouser Price/Stock" "https://www.mouser.co.uk/ProductDetail/Vishay-Semiconductors/SI2302DDS-T1-GE3?qs=MxnWX8BLHKdaCSNWhg%252BxLA%3D%3D" (at 127 768.91 0)
-      (effects (font (size 1.27 1.27)) (justify left top) hide)
-    )
-    (property "Manufacturer_Name" "Vishay" (at 127 868.91 0)
-      (effects (font (size 1.27 1.27)) (justify left top) hide)
-    )
-    (property "Manufacturer_Part_Number" "SI2302DDS-T1-GE3" (at 127 968.91 0)
+    (property "Reference" "Q8" (at 99.06 59.69 0)
+      (effects (font (size 1.27 1.27)) (justify left))
+    )
+    (property "Value" "SI2302DDS-T1-GE3" (at 99.06 62.23 0)
+      (effects (font (size 1.27 1.27)) (justify left))
+    )
+    (property "Footprint" "footprints:SI2302DDS-T1-GE3" (at 104.14 104.14 0)
+      (effects (font (size 1.27 1.27)) (justify left top) hide)
+    )
+    (property "Datasheet" "http://www.vishay.com/docs/63653/si2302dds.pdf" (at 91.186 106.934 0)
+      (effects (font (size 1.27 1.27)) (justify left top) hide)
+    )
+    (property "Height" "1.12" (at 127 468.58 0)
+      (effects (font (size 1.27 1.27)) (justify left top) hide)
+    )
+    (property "Mouser Part Number" "78-SI2302DDS-T1-GE3" (at 127 568.58 0)
+      (effects (font (size 1.27 1.27)) (justify left top) hide)
+    )
+    (property "Mouser Price/Stock" "https://www.mouser.co.uk/ProductDetail/Vishay-Semiconductors/SI2302DDS-T1-GE3?qs=MxnWX8BLHKdaCSNWhg%252BxLA%3D%3D" (at 127 668.58 0)
+      (effects (font (size 1.27 1.27)) (justify left top) hide)
+    )
+    (property "Manufacturer_Name" "Vishay" (at 127 768.58 0)
+      (effects (font (size 1.27 1.27)) (justify left top) hide)
+    )
+    (property "Manufacturer_Part_Number" "SI2302DDS-T1-GE3" (at 127 868.58 0)
       (effects (font (size 1.27 1.27)) (justify left top) hide)
     )
@@
       (project "eps-re_project"
         (path "/2eebaa11-d7ed-4bfd-bc8e-988f68654d29/6f34948c-43a8-4614-b8ed-90c5b6b9b243"
-          (reference "Q2") (unit 1)
-        )
-        (path "/2eebaa11-d7ed-4bfd-bc8e-988f68654d29/6cd5fe02-9b19-49bf-9109-b0a2c2f10c14"
-          (reference "Q2") (unit 1)
+          (reference "Q8") (unit 1)
+        )
+        (path "/2eebaa11-d7ed-4bfd-bc8e-988f68654d29/6cd5fe02-9b19-49bf-9109-b0a2c2f10c14"
+          (reference "Q1") (unit 1)
         )
       )
@@
         )
       )
+    )
+  )
+  (symbol (lib_id "SI2302DDS-T1-GE3:SI2302DDS-T1-GE3") (at 115.57 170.18 0) (unit 1)
+    (in_bom yes) (on_board yes) (dnp no)
+    (property "Reference" "Q8" (at 99.06 160.02 0)
+      (effects (font (size 1.27 1.27)) (justify left))
+    )
+    (property "Value" "SI2302DDS-T1-GE3" (at 99.06 162.56 0)
+      (effects (font (size 1.27 1.27)) (justify left))
+    )
+    (property "Footprint" "footprints:SI2302DDS-T1-GE3" (at 104.14 204.47 0)
+      (effects (font (size 1.27 1.27)) (justify left top) hide)
+    )
+    (property "Datasheet" "http://www.vishay.com/docs/63653/si2302dds.pdf" (at 91.186 207.264 0)
+      (effects (font (size 1.27 1.27)) (justify left top) hide)
+    )
+    (property "Height" "1.12" (at 127 568.91 0)
+      (effects (font (size 1.27 1.27)) (justify left top) hide)
+    )
+    (property "Mouser Part Number" "78-SI2302DDS-T1-GE3" (at 127 668.91 0)
+      (effects (font (size 1.27 1.27)) (justify left top) hide)
+    )
+    (property "Mouser Price/Stock" "https://www.mouser.co.uk/ProductDetail/Vishay-Semiconductors/SI2302DDS-T1-GE3?qs=MxnWX8BLHKdaCSNWhg%252BxLA%3D%3D" (at 127 768.91 0)
+      (effects (font (size 1.27 1.27)) (justify left top) hide)
+    )
+    (property "Manufacturer_Name" "Vishay" (at 127 868.91 0)
+      (effects (font (size 1.27 1.27)) (justify left top) hide)
+    )
+    (property "Manufacturer_Part_Number" "SI2302DDS-T1-GE3" (at 127 968.91 0)
+      (effects (font (size 1.27 1.27)) (justify left top) hide)
+    )
+    (pin "1")
+    (pin "2")
+    (pin "3")
+    (instances
+      (project "eps-re_project"
+        (path "/2eebaa11-d7ed-4bfd-bc8e-988f68654d29/6f34948c-43a8-4614-b8ed-90c5b6b9b243"
+          (reference "Q8") (unit 1)
+        )
+        (path "/2eebaa11-d7ed-4bfd-bc8e-988f68654d29/6cd5fe02-9b19-49bf-9109-b0a2c2f10c14"
+          (reference "Q2") (unit 1)
+        )
+      )

Commit message: hardware: Updating 3D models, component placement and more.
Other:
- title: (none) -> Reliability Enhanced Electrical Power System
Changed lines of the file:
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@@
 (kicad_sch (version 20230121) (generator eeschema)
   (paper "A3")
+  (title_block
+    (title "Reliability Enhanced Electrical Power System")
+    (date "2023-08-03")
+    (rev "v0.0")
+    (comment 1 "João C. E. Barcellos <joaoclaudiobarcellos@gmail.com>")
+    (comment 2 "Laura Debastiani <laudebastiani@gmail.com>")
+  )
   (junction (at 74.93 170.18) (diameter 0) (color 0 0 0 0)
   )
