File: hardware/House_Keeping.kicad_sch (KiCad schematic)
At the start: 4 parts, among them Q7 SI2302DDS-T1-GE3, U15 CD4051BPWR, U16 CD4051BPWR

Commit message: hardware: update schematic and layout projects
Other:
- moved on the sheet: Q7, R1
