File: hardware/eps-re_project.kicad_sch (KiCad schematic)
At the start: 50 parts, among them J1 2053380004, J13 533980671, J14 533980471, J2 2053380004, J21 2053380002, J22 2053380002, J25 2053380002, J26 2053380002, J27 2053380002, J28 2053380002, J29 2053380002, J3 533980471, J4 2053380004, J5 533980471, J6 533980471, J7 533980471

Commit message: hardware: update schematic and layout projects
Parts:
- removed J13: 533980671, footprints:533980671, symbol 533980671:53398-0671
- removed J14, J3, J5, J6, J7: 533980471, footprints:533980471, symbol 533980471:533980471
- added J13: 532610671, footprints:532610671, symbol 532610671:532610671
- added J3, J5, J6, J7, J8: 532610471, footprints:532610471, symbol 532610471:532610471
- D17, D18, D19, D20, D21, D22: Package US2H-2 -> SOD-323HE
- J1, J2, J4: Package Pico-Lock (4P) -> N/A
- J21, J22, J25, J26, J27, J28, J29: Package Pico-Lock (2P) -> N/A
- renumbered TP2 to TP10, TP2 to TP11, TP2 to TP12, TP2 to TP13, TP2 to TP14, TP2 to TP15, TP2 to TP16, TP2 to TP17, TP2 to TP18, TP2 to TP19, TP2 to TP20, TP2 to TP21, TP2 to TP22, TP2 to TP23, TP2 to TP24, TP2 to TP25, TP2 to TP26, TP2 to TP27, TP2 to TP3, TP2 to TP7, TP2 to TP8, TP2 to TP9
Connections:
- net 3V3_A_~{EN}: now also J3.2
- net 3V3_B_~{EN}: now also J5.1
- net 5V0_A_~{EN}: now also J3.3
- net 5V0_B_~{EN}: now also J5.3
- net AMUX_OUT: now also J13.5
- net AMUX_SEL0: now also J13.2
- net AMUX_SEL1: now also J13.3
- net AMUX_SEL2: now also J13.4
- net AMUX_SEL3: now also J13.1
- net AntDep_EN: now also J7.4
- net BC_A_TS: now also J8.3
- net BC_A_~{EN}: now also J3.1
- net BC_B_TS: now also J8.2
- net BC_B_~{EN}: now also J5.2
- net BC_VFB: now also J8.1
- net Beacon_EN: now also J7.3
- net GNDPWR: now also J13.6, J3.4, J5.4, J6.4, J7.1, J8.4
- net OBDH_EN: now also J7.2
- net Payload_EN: now also J6.3
- net RadioBeacon_EN: now also J6.2
- net RadioMain_EN: now also J6.1
Other:
- note removed: "ANALOG SIGNALS"
- note removed: "Authors"
- note removed: "BLOCK DIAGRAM"
- note removed: "MOUNTING HOLES"
- note removed: "Modifications"
- note removed: "POWER FLAGS"
- note removed: "REVISION HISTORY"
- note removed: "TEST POINTS"
- note removed: "Version"
- moved on the sheet: D17, D18, D19, D20, D21, D22, H1, H2, H3, H4, J1, J2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
